Commit message: Solution to exercise 2.0

File: urdf/mira_simple_collisions_inertias.urdf (robot description, URDF)
Before this commit: robot mira, 2 links, 1 joints
Links:
- link base_link: mass None -> 0.18; geometry collision cylinder length=0.09 radius=0.06; visual cylinder length=0.09 radius=0.06
- link roll_M1_link: mass None -> 0.001; geometry visual cylinder length=0.005 radius=0.01
